File: Schematics/IFE_DISPLAY/Display_Board.sch (EAGLE design)
At the start: 76 parts, among them IC2 EP2C5T144, Q1 16MHz, Q2 MMBT3904L, U1 MCP1826S-1802E/DB, U10 TPS5420D, U2 EPCS1SI8N, U3 ATMEGA328P-AU, U4 HEX_CONVERTER, U5 HEX_CONVERTER, U9 TPS5420D, X3 16MHz

Commit message: Initial board organization. Time to route
Parts:
- removed X3: 16MHz, crystal:CRYSTAL
- added Q3: 16MHz, adafruit:CRYSTALCTS406
- R35: value 5.9k -> 3.2k
Connections:
- removed net GREEN_8: IC2.IO51
- net BLUE_0: now also IC2.IO40; no longer IC2.IO52
- net BLUE_1: now also IC2.IO32; no longer IC2.IO53
- net BLUE_2: now also IC2.IO31; no longer IC2.IO55
- net BLUE_3: now also IC2.IO30; no longer IC2.IO57
- net BLUE_4: now also IC2.IO28; no longer IC2.IO58
- net BLUE_5: now also IC2.IO27; no longer IC2.IO59
- net BLUE_6: now also IC2.IO26; no longer IC2.IO60
- net BLUE_7: now also IC2.IO25; no longer IC2.IO63
- net DISP_CLK: now also IC2.IO9; no longer IC2.IO3
- net DISP_DEN: now also IC2.IO3; no longer IC2.IO9
- net DISP_EN: now also IC2.IO8; no longer IC2.IO4
- net DISP_VSYNC: now also IC2.IO4; no longer IC2.IO8
- net GREEN_0: now also IC2.IO51; no longer IC2.IO41
- net GREEN_1: now also IC2.IO48; no longer IC2.IO42
- net GREEN_2: now also IC2.IO47; no longer IC2.IO43
- net GREEN_3: now also IC2.IO45
- net GREEN_5: now also IC2.IO43; no longer IC2.IO45
- net GREEN_6: now also IC2.IO42; no longer IC2.IO47
- net GREEN_7: now also IC2.IO41; no longer IC2.IO48
- net RED_0: now also IC2.IO63; no longer IC2.IO25
- net RED_1: now also IC2.IO60; no longer IC2.IO26
- net RED_2: now also IC2.IO59; no longer IC2.IO27
- net RED_3: now also IC2.IO58; no longer IC2.IO28
- net RED_4: now also IC2.IO57; no longer IC2.IO30
- net RED_5: now also IC2.IO55; no longer IC2.IO31
- net RED_6: now also IC2.IO53; no longer IC2.IO32
- net RED_7: now also IC2.IO52; no longer IC2.IO40
- net XTAL1: now also Q3.2; no longer X3.2
- net XTAL2: now also Q3.1; no longer X3.1

Commit message: Layout started
Changed lines of the file:
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@@
 <pinref part="GND19" gate="1" pin="GND"/>
 <wire x1="294.64" y1="91.44" x2="294.64" y2="88.9" width="0.1524" layer="91"/>
+<junction x="294.64" y="91.44"/>
+<junction x="289.56" y="91.44"/>
 </segment>
 <segment>
@@
 <wire x1="167.64" y1="30.48" x2="162.56" y2="30.48" width="0.1524" layer="91"/>
 <wire x1="167.64" y1="35.56" x2="167.64" y2="30.48" width="0.1524" layer="91"/>
+<junction x="167.64" y="30.48"/>
 </segment>
 <segment>
@@
 <wire x1="312.42" y1="25.4" x2="312.42" y2="22.86" width="0.1524" layer="91"/>
 <wire x1="299.72" y1="25.4" x2="312.42" y2="25.4" width="0.1524" layer="91"/>
+<junction x="312.42" y="25.4"/>
 </segment>
 <segment>
@@
 <wire x1="243.84" y1="25.4" x2="243.84" y2="22.86" width="0.1524" layer="91"/>
 <wire x1="226.06" y1="25.4" x2="243.84" y2="25.4" width="0.1524" layer="91"/>
+<junction x="243.84" y="25.4"/>
 </segment>
 </net>
@@
 </sheet>
 </sheets>
+<errors>
+</errors>
 </schematic>
 </drawing>

Commit message: More optimizations and working on interconnect for display board
Connections:
- net BLUE_0: now also IC2.IO52; no longer IC2.IO40
- net BLUE_1: now also IC2.IO53; no longer IC2.IO32
- net BLUE_2: now also IC2.IO55; no longer IC2.IO31
- net BLUE_3: now also IC2.IO57; no longer IC2.IO30
- net BLUE_4: now also IC2.IO58; no longer IC2.IO28
- net BLUE_5: now also IC2.IO59; no longer IC2.IO27
- net BLUE_6: now also IC2.IO60; no longer IC2.IO26
- net BLUE_7: now also IC2.IO63; no longer IC2.IO25
- net DISP_CLK: now also IC2.IO3; no longer IC2.IO9
- net DISP_DEN: now also IC2.IO9; no longer IC2.IO3
- net DISP_EN: now also IC2.IO4; no longer IC2.IO8
- net DISP_VSYNC: now also IC2.IO8; no longer IC2.IO4
- net FPGA_D0_3_3: now also IC2.IO75; no longer IC2.IO142
- net FPGA_D1_3_3: now also IC2.IO76; no longer IC2.IO141
- net FPGA_D2_3_3: now also IC2.IO79; no longer IC2.IO139
- net FPGA_D3_3_3: now also IC2.IO80; no longer IC2.IO137
- net FPGA_R0_3_3: now also IC2.IO81; no longer IC2.IO136
- net FPGA_R1_3_3: now also IC2.IO86; no longer IC2.IO135
- net FPGA_R2_3_3: now also IC2.IO87; no longer IC2.IO134
- net FPGA_R3_3_3: now also IC2.IO92; no longer IC2.IO133
- net FPGA_RSEL_3_3: now also IC2.IO73; no longer IC2.IO144
- net FPGA_W_3_3: now also IC2.IO74; no longer IC2.IO143
- net GREEN_0: now also IC2.IO41; no longer IC2.IO51
- net GREEN_1: now also IC2.IO42; no longer IC2.IO48
- net GREEN_2: now also IC2.IO43; no longer IC2.IO47
- net GREEN_3: now also IC2.IO44; no longer IC2.IO45
- net GREEN_4: now also IC2.IO45; no longer IC2.IO44
- net GREEN_5: now also IC2.IO47; no longer IC2.IO43
- net GREEN_6: now also IC2.IO48; no longer IC2.IO42
- net GREEN_7: now also IC2.IO51; no longer IC2.IO41
- net RED_0: now also IC2.IO25; no longer IC2.IO63
- net RED_1: now also IC2.IO26; no longer IC2.IO60
- net RED_2: now also IC2.IO27; no longer IC2.IO59
- net RED_3: now also IC2.IO28; no longer IC2.IO58
- net RED_4: now also IC2.IO30; no longer IC2.IO57
- net RED_5: now also IC2.IO31; no longer IC2.IO55
- net RED_6: now also IC2.IO32; no longer IC2.IO53
- net RED_7: now also IC2.IO40; no longer IC2.IO52

Commit message: added 120 ohm resistor
Parts:
- added R1: 120, rcl:R-US_R0805
Connections:
- net CANH: now also R1.1
- net CANL: now also R1.2
Changed lines of the file:
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@@
 <?xml version="1.0" encoding="utf-8"?>
 <!DOCTYPE eagle SYSTEM "eagle.dtd">
-<eagle version="8.4.1">
+<eagle version="8.4.0">
 <drawing>
 <settings>
@@
 <part name="FRAME3" library="frames" library_urn="urn:adsk.eagle:library:229" deviceset="A3L-LOC" device=""/>
 <part name="Q3" library="adafruit" deviceset="CRYSTAL" device="CTS406" value="16MHz"/>
+<part name="R1" library="rcl" deviceset="R-US_" device="R0805" value="120"/>
 </parts>
 <sheets>
@@
 <instance part="FRAME2" gate="G$1" x="-27.94" y="-66.04"/>
 <instance part="Q3" gate="G$1" x="172.72" y="15.24" rot="R90"/>
+<instance part="R1" gate="G$1" x="294.64" y="127" rot="R180"/>
 </instances>
 <busses>
@@
 <wire x1="289.56" y1="116.84" x2="289.56" y2="121.92" width="0.1524" layer="91"/>
 <junction x="289.56" y="121.92"/>
+<pinref part="R1" gate="G$1" pin="2"/>
+<wire x1="289.56" y1="121.92" x2="289.56" y2="127" width="0.1524" layer="91"/>
 </segment>
 <segment>
@@
 <wire x1="299.72" y1="116.84" x2="299.72" y2="119.38" width="0.1524" layer="91"/>
 <junction x="299.72" y="119.38"/>
-</segment>
-<segment>
+<pinref part="R1" gate="G$1" pin="1"/>
+<wire x1="299.72" y1="127" x2="299.72" y2="119.38" width="0.1524" layer="91"/>
+</segment>
+<segment>

Commit message: Redid the Switching Supplies
Parts:
- removed C25: 0.1u, rcl:C-EUC0805K
- removed C26, C33: 4.7uF, resistor:C-EUC0805K
- removed C27, C34: 0.01uF, resistor:C-EUC0805K
- removed C28, C29, C35, C36: 47uF, rcl:C-EUC0805K
- removed C30, C37: 1800pF, rcl:C-EUC0805K
- removed C31, C38: 0.1uF, rcl:C-EUC0805K
- removed C32, C39: 150pF, rcl:C-EUC0805K
- removed C40: 220u, Capacitors:C1206
- removed D4, D5: (no value), adafruit:DIODESMA
- removed FUSE4: MINI297-3568, Fuse:MINI297-3568
- removed L6: 23uH, Inductors:MSS7348
- removed L7: 58uH, Inductors:MSS7348
- removed L8: 20uH, Inductors:MSS7348
- removed Q2: MMBT3904L, transistor-npn:BCW31SMD
- removed R12: 5.9k, rcl:R-US_R0805
- removed R13, R36: 549, rcl:R-US_R0805
- removed R25: 76, resistor:R-US_R0805
- removed R26: 5.2k, resistor:R-US_R0805
- removed R34: 10k, rcl:R-US_R0805
- removed R35: 3.2k, rcl:R-US_R0805
- removed U1: MCP1826S-1802E/DB, Microchip_By_element14_Batch_1:MCP1826S-1802E/DB
- removed U10, U9: TPS5420D, Texas Instruments_By_element14_Batch_1:TPS5420D
- added C1, C2: 1uF, rcl:C-EUC0805K
- added C10, C11, C12, C5: 0.1u, rcl:C-EUC0805K
- added C13: 10uF, microbuilder:CAP_CERAMIC_0805MP
- added C14, C16: 1uF, microbuilder:CAP_CERAMIC_0805MP
- added C15: 0.1uF, microbuilder:CAP_CERAMIC_0805MP
- added D2: MBR0540, microbuilder:DIODESOD-123
- added D3: MM3Z24VT1G, microbuilder:DIODESMA
- added L1: 6.8uH power L CID 2276, microbuilder:INDUCTORNR5040
- added R11: 6Ω, microbuilder:RESISTOR_0805MP
- added R2: 12Ω, microbuilder:RESISTOR_0805MP
- added U$5: MCP1702T-1202E/CB, Microchip_By_element14_Batch_1:MCP1702T-1802E/CB
- added U6: MC78LC33NTRG, ON Semiconductor_By_element14_Batch_1:MC78LC33NTRG
- added U7: MC78LC50NTRG, ON Semiconductor_By_element14_Batch_1:MC78LC50NTRG
- added U8: FAN5333BSX, microbuilder:FAN5331
- R3: value 10k -> 10K; device rcl:R-US_R0805 -> microbuilder:RESISTOR_0805MP
Connections:
- removed net +24V: C40.1, L8.2, R25.2
- removed net N$13: Q2.B, R26.1
- removed net N$22: C27.1, U9.BOOT
- removed net N$23: C27.2, D4.C, L6.1, U9.PH
- removed net N$25: C30.2, C31.1, C32.1, R12.2, R3.1, U9.VSENSE
- removed net N$26: C31.2, R13.2
- removed net N$27: C34.1, U10.BOOT
- removed net N$28: C34.2, D5.C, L7.1, U10.PH
- removed net N$30: C37.2, C38.1, C39.1, R34.1, R35.2, U10.VSENSE
- removed net N$31: C38.2, R36.2
- removed net N$32: FUSE4.1, L8.1
- new net N$8: D2.A, L1.2, U8.SW
- net +12V: now also C10.1, C11.1, C2.1, U$5.VIN, U6.VIN, U7.VIN; no longer C26.1, C33.1, U10.ENA, U10.VIN, U9.ENA, U9.VIN
- net +3V3: now also C12.1, U6.VOUT; no longer C28.1, C29.1, C30.1, L6.2, R3.2, U1.VIN
- net +5V: now also C13.1, C5.1, L1.1, R3.2, U7.VOUT, U8.VIN; no longer C35.1, C36.1, C37.1, L7.2, R34.2
- net DISP_LEDA: now also C14.1, C16.1, D2.C, D3.C; no longer R25.1
- net DISP_LEDK: now also C15.1, D3.A, R11.2, R2.2, U8.FB; no longer Q2.C
- net DISP_PWM: now also R3.1, U8.SHDN; no longer R26.2
- net GND: now also C1.2, C10.2, C11.2, C12.2, C13.2, C14.2, C15.2, C16.2, C2.2, C5.2, R11.1, R2.1, U$5.GND, U6.GND, U7.GND, U8.GND; no longer C25.2, C26.2, C28.2, C29.2, C32.2, C33.2, C35.2, C36.2, C39.2, C40.2, D4.A, D5.A, Q2.E, R12.1, R13.1, R35.1, R36.1, U1.GND_(TAB), U1.GND_(TAB)_2, U10.GND, U9.GND
- net PWR_IN_24: no longer FUSE4.2
- net VCC: now also C1.1, U$5.VOUT; no longer C25.1, U1.VOUT
Other:
- note removed: "Display PWM Circuitry"

Commit message: Finishing up hardware portion of report
Other:
- note removed: "CAN Tranciever (MCP 2551)"
- moved on the sheet: C24, C3, C4, C6, C7, C8, C9, D1, FUSE3, JP1, L5, LED1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
