File: Schematics/IFE_DISPLAY/Display_Board_v2.brd (EAGLE design)
At the start: 96.5 x 83.8 mm, 79 parts, among them U4 HEX_CONVERTER, U5 HEX_CONVERTER

Commit message: Made a few custom parts
Parts:
- L1: value 6.8uH -> 10uH
Changed lines of the file:
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@@
 <?xml version="1.0" encoding="utf-8"?>
 <!DOCTYPE eagle SYSTEM "eagle.dtd">
-<eagle version="8.6.0">
+<eagle version="8.7.0">
 <drawing>
 <settings>
@@
 <attribute name="VALUE" x="5.08" y="71.755" size="1.27" layer="27"/>
 </element>
-<element name="L1" library="microbuilder" package="INDUCTOR_5X5MM_NR5040_NOTHERMALS" value="6.8uH" x="44.45" y="74.93" smashed="yes" rot="R270">
+<element name="L1" library="microbuilder" package="INDUCTOR_5X5MM_NR5040_NOTHERMALS" value="10uH" x="44.45" y="74.93" smashed="yes" rot="R270">
 <attribute name="NAME" x="42.9002" y="79.0182" size="0.8128" layer="25" font="vector" rot="R180"/>
 </element>
