File: Schematics/IFE_DISPLAY/Display_Board_v3.brd (EAGLE design)
At the start: 96.5 x 83.8 mm, 73 parts, among them IC2 EP2C5T144, U2 EPCS1SI8N, U4 HEX_CONVERTER, U5 HEX_CONVERTER

Commit message: V3 Under Review
Connections:
- net LED2: no longer IC2.132
Routing:
- net +3V3: track 227.1 -> 380.9 mm, vias 7 -> 16
- net GND: track 4.67 -> 132.7 mm, vias 0 -> 18
- net VCC: track 17.2 -> 113.5 mm, vias 2 -> 6
- net DISP_PWM: track 8.28 -> 89.0 mm, vias 1 -> 6
- net +5V: track 147.3 -> 185.5 mm, vias 4 -> 9
