File: Schematics/IFE_DISPLAY/Display_Board_v3.sch (EAGLE design)
At the start: 73 parts, among them IC2 EP2C5T144, U2 EPCS1SI8N, U4 HEX_CONVERTER, U5 HEX_CONVERTER

Commit message: V3 Under Review
Connections:
- net LED2: no longer IC2.IO132
Other:
- note removed: "DC-DC Power Converter"
- moved on the sheet: 1.2T, 3.3T, 5T, AS1, C1, C10, C11, C12, C13, C16, C17, C18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
