File: Schematics/IFE_DISPLAY/Display_Board_v4.brd (EAGLE design)
At the start: 96.5 x 83.8 mm, 59 parts, among them J1 5.5x2.1mm Barrel, Q2 2N7002PW, U1 FT231XS

Commit message: Added 2 new power relays
Parts:
- C3, C4, C6, C7: value 22p -> 18p
- R12, R13: value 1k -> 330
- RX: value Yellow -> RED
- TX: value Red -> RED
- U$15: value 406CYRYSTAL -> 16MHz
Changed lines of the file:
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@@
 <attribute name="VALUE" x="50.4444" y="11.7856" size="2.0828" layer="27" ratio="10" rot="SR90"/>
 </element>
-<element name="C3" library="resistor" package="C0805K" value="22p" x="53.34" y="6.35" smashed="yes" rot="R270">
+<element name="C3" library="resistor" package="C0805K" value="18p" x="53.34" y="6.35" smashed="yes" rot="R270">
 <attribute name="NAME" x="51.2686" y="5.6736" size="0.8128" layer="25" rot="R270"/>
 </element>
-<element name="C4" library="resistor" package="C0805K" value="22p" x="63.5" y="6.35" smashed="yes" rot="R270">
+<element name="C4" library="resistor" package="C0805K" value="18p" x="63.5" y="6.35" smashed="yes" rot="R270">
 <attribute name="NAME" x="64.7814" y="5.6736" size="0.8128" layer="25" rot="R270"/>
 </element>
-<element name="C6" library="resistor" package="C0805K" value="22p" x="69.85" y="13.97" smashed="yes">
+<element name="C6" library="resistor" package="C0805K" value="18p" x="69.85" y="13.97" smashed="yes">
 <attribute name="NAME" x="68.088" y="14.9974" size="0.8128" layer="25"/>
 </element>
-<element name="C7" library="resistor" package="C0805K" value="22p" x="69.85" y="3.81" smashed="yes">
+<element name="C7" library="resistor" package="C0805K" value="18p" x="69.85" y="3.81" smashed="yes">
 <attribute name="NAME" x="67.961" y="4.939" size="0.8128" layer="25"/>
 </element>
@@
 <attribute name="NAME" x="61.849" y="8.5852" size="0.8128" layer="25" rot="R270"/>
 </element>
-<element name="U$15" library="Display_Custom" package="CTS406" value="406CYRYSTAL" x="69.85" y="8.89" smashed="yes" rot="R270">
+<element name="U$15" library="Display_Custom" package="CTS406" value="16MHz" x="69.85" y="8.89" smashed="yes" rot="R270">
 <attribute name="NAME" x="67.5894" y="12.2936" size="0.8128" layer="25"/>
 </element>
@@
 <attribute name="NAME" x="46.99" y="24.765" size="0.8128" layer="25" rot="R90"/>
 </element>
-<element name="R12" library="SparkFun-Resistors" package="0603" value="1k" x="35.56" y="76.2" smashed="yes" rot="MR0">
+<element name="R12" library="SparkFun-Resistors" package="0603" value="330" x="35.56" y="76.2" smashed="yes" rot="MR0">
 <attribute name="NAME" x="35.56" y="77.0128" size="0.6096" layer="26" font="vector" ratio="20" rot="MR0" align="bottom-center"/>
 <attribute name="PROD_ID" value="RES-07856" x="41.91" y="93.98" size="1.778" layer="28" rot="MR0" display="off"/>
 </element>
-<element name="R13" library="SparkFun-Resistors" package="0603" value="1k" x="35.56" y="73.66" smashed="yes" rot="MR0">
+<element name="R13" library="SparkFun-Resistors" package="0603" value="330" x="35.56" y="73.66" smashed="yes" rot="MR0">
 <attribute name="NAME" x="35.56" y="74.5744" size="0.6096" layer="26" font="vector" ratio="20" rot="MR0" align="bottom-center"/>
 <attribute name="PROD_ID" value="RES-07856" x="48.26" y="87.63" size="1.778" layer="28" rot="MR0" display="off"/>
@@
 <attribute name="PROD_ID" value="CAP-00810" x="22.8854" y="103.6066" size="1.778" layer="28" rot="MR180" display="off"/>
 </element>
-<element name="RX" library="SparkFun-LED" package="LED-1206" value="Yellow" x="30.48" y="73.66" smashed="yes" rot="MR0">
+<element name="RX" library="SparkFun-LED" package="LED-1206" value="RED" x="30.48" y="73.66" smashed="yes" rot="MR0">
 <attribute name="NAME" x="30.4546" y="71.9963" size="0.6096" layer="26" font="vector" ratio="20" rot="MR0" align="bottom-center"/>
 <attribute name="PROD_ID" value="DIO-09909" x="62.23" y="29.21" size="1.778" layer="28" rot="MR0" display="off"/>
 </element>
-<element name="TX" library="SparkFun-LED" package="LED-1206" value="Red" x="30.48" y="76.2" smashed="yes" rot="MR0">
+<element name="TX" library="SparkFun-LED" package="LED-1206" value="RED" x="30.48" y="76.2" smashed="yes" rot="MR0">
 <attribute name="NAME" x="30.48" y="77.3811" size="0.6096" layer="26" font="vector" ratio="20" rot="MR0" align="bottom-center"/>
 <attribute name="PROD_ID" value="DIO-09912" x="62.23" y="31.75" size="1.778" layer="28" rot="MR0" display="off"/>
